Commit message: Pose, Wr, Wl listos

File: urdf/puzzle_bot.urdf (robot description, URDF)
Before this commit: robot puzzle_drone, 4 links, 3 joints
Links:
- link base_link: geometry visual mesh filename=package://reto_sem_3/meshes/Puzzlebot_Jetson_Lidar_Edition_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
- link caster_link: geometry visual mesh filename=package://reto_sem_3/meshes/Puzzlebot_Caster_Wheel.stl
- link wheel_l_link: geometry visual mesh filename=package://reto_sem_3/meshes/Puzzlebot_Wheel.stl
- link wheel_r_link: geometry visual mesh filename=package://reto_sem_3/meshes/Puzzlebot_Wheel.stl

Commit message: elipsoide creada

File: urdf/puzzle_bot.urdf (robot description, URDF)
Before this commit: robot puzzle_bot, 4 links, 3 joints
Links:
- link base_link: geometry visual mesh filename=package://reto_sem_5/meshes/Puzzlebot_Jetson_Lidar_Edition_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
- link caster_link: geometry visual mesh filename=package://reto_sem_5/meshes/Puzzlebot_Caster_Wheel.stl
- link wheel_l_link: geometry visual mesh filename=package://reto_sem_5/meshes/Puzzlebot_Wheel.stl
- link wheel_r_link: geometry visual mesh filename=package://reto_sem_5/meshes/Puzzlebot_Wheel.stl

Commit message: Se separo point generator en su proprio nodo y se empezo añadir los namespaces del reto anterior

File: urdf/puzzle_bot.urdf (robot description, URDF)
Before this commit: robot puzzle_bot, 4 links, 3 joints
Links:
- link base_link: geometry visual mesh filename=package://reto_sem_6/meshes/Puzzlebot_Jetson_Lidar_Edition_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
- link caster_link: geometry visual mesh filename=package://reto_sem_6/meshes/Puzzlebot_Caster_Wheel.stl
- link wheel_l_link: geometry visual mesh filename=package://reto_sem_6/meshes/Puzzlebot_Wheel.stl
- link wheel_r_link: geometry visual mesh filename=package://reto_sem_6/meshes/Puzzlebot_Wheel.stl
